Commit message: Update to arm dimensions
Thanks Yasamin!

File: r3ros/arm-urdf/arm-sample.urdf (robot description, URDF)
Before this commit: robot cougarbot, 6 links, 5 joints
Links:
- link lower_arm: geometry collision cylinder length=0.4 radius=0.05; visual cylinder length=0.4 radius=0.05
- link torso: geometry collision cylinder length=0.5 radius=0.05; visual cylinder length=0.5 radius=0.05
- link upper_arm: geometry collision cylinder length=0.4 radius=0.05; visual cylinder length=0.4 radius=0.05
Joints:
- joint elbow: origin xyz=0.0 0.1 0.5063 rpy=0 0 0 -> xyz=0.0 0.1 0.35 rpy=0 0 0
- joint shoulder: origin xyz=0.0 -0.1 0.084 rpy=0 1.5708 0 -> xyz=0.0 -0.1 0.45 rpy=0 1.5708 0
- joint wrist: origin xyz=0.0 0.0 0.39 rpy=0 0 0 -> xyz=0.0 0.0 0.425 rpy=0 0 0
