Commit message: Update robot.urdf

File: r3ros/urdf/robot.urdf (robot description, URDF)
Before this commit: robot tortoisebot, 6 links, 5 joints
Links:
- added link bl_wheel, mass 0.1; collision cylinder length=0.1 radius=0.127; visual cylinder length=0.10 radius=0.127
Joints:
- added joint back_left_wheelconnect: type continuous, parent base_link, child bl_wheel, origin xyz=0.3 0 0, axis 0 0 1

Commit message: Revert "Update robot.urdf"
This reverts commit 317d93cc44d69eaa5f2ab7f0f7c01dce68240f1b.

File: r3ros/urdf/robot.urdf (robot description, URDF)
Before this commit: robot tortoisebot, 7 links, 6 joints
Links:
- removed link bl_wheel
Joints:
- removed joint back_left_wheelconnect
