Commit message: Update test_design.urdf

File: r3ros/urdf/test_design.urdf (robot description, URDF)
Before this commit: robot cougarbot, 2 links, 1 joints
Joints:
- joint base_to_right_leg: origin xyz=0.22 0 .25 -> xyz=.16 1.29 0

Commit message: Update test_design.urdf

File: r3ros/urdf/test_design.urdf (robot description, URDF)
Before this commit: robot cougarbot, 2 links, 1 joints
Joints:
- joint base_to_right_leg: origin xyz=.16 1.29 0 -> xyz=0 1.29 0

Commit message: Update test_design.urdf

File: r3ros/urdf/test_design.urdf (robot description, URDF)
Before this commit: robot cougarbot, 2 links, 1 joints
Joints:
- removed joint base_to_right_leg
- added joint front_left_wheelconnect: type fixed, parent base_link, child fl_wheel, origin xyz=0 0.645 0

Commit message: Update test_design.urdf

File: r3ros/urdf/test_design.urdf (robot description, URDF)
Before this commit: robot cougarbot, 2 links, 1 joints
Links:
- added link front_wheel_left_axel; visual box size=0.3 .1 0.06
Joints:
- joint front_left_wheelconnect: origin xyz=0 0.645 0 -> xyz=-0.08 -.645 0; parent base_link -> front_wheel_left_axel

Commit message: Update test_design.urdf

File: r3ros/urdf/test_design.urdf (robot description, URDF)
Before this commit: robot cougarbot, 3 links, 1 joints
Joints:
- added joint front_left_jointconnect: type fixed, parent base_link, child front_wheel_left_axel, origin xyz=-0.08 -.645 0

Commit message: Update test_design.urdf

File: r3ros/urdf/test_design.urdf (robot description, URDF)
Before this commit: robot cougarbot, 3 links, 2 joints
Joints:
- joint front_left_wheelconnect: origin xyz=-0.08 -.645 0 -> xyz=0 0 0

Commit message: Update test_design.urdf

File: r3ros/urdf/test_design.urdf (robot description, URDF)
Before this commit: robot cougarbot, 3 links, 2 joints
Links:
- added link back_wheel_left_axel; visual box size=0.3 .1 0.06
- added link middle_wheel_left_axel; visual box size=0.3 .1 0.06
- link base_link: geometry visual box size=0.16 1.057 0.12

Commit message: Update test_design.urdf

File: r3ros/urdf/test_design.urdf (robot description, URDF)
Before this commit: robot cougarbot, 5 links, 2 joints
Joints:
- added joint back_left_jointconnect: type fixed, parent base_link, child back_wheel_left_axel, origin xyz=0.08 1.057 0
- added joint middle_left_jointconnect: type fixed, parent base_link, child middle_wheel_left_axel, origin xyz=0.08 0.5285 0

Commit message: Update test_design.urdf

File: r3ros/urdf/test_design.urdf (robot description, URDF)
Before this commit: robot cougarbot, 5 links, 4 joints
Joints:
- joint front_left_jointconnect: origin xyz=-0.08 -.645 0 -> xyz=0.08 0.645 0

Commit message: Update test_design.urdf

File: r3ros/urdf/test_design.urdf (robot description, URDF)
Before this commit: robot cougarbot, 5 links, 4 joints
Joints:
- joint front_left_jointconnect: origin xyz=0.08 0.645 0 -> xyz=0.08 0 0

Commit message: Update test_design.urdf

File: r3ros/urdf/test_design.urdf (robot description, URDF)
Before this commit: robot cougarbot, 5 links, 4 joints
Joints:
- joint back_left_jointconnect: origin xyz=0.08 1.057 0 -> xyz=0.15 0.5285 0
- joint front_left_jointconnect: origin xyz=0.08 0 0 -> xyz=0.15 -0.5285 0
- joint middle_left_jointconnect: origin xyz=0.08 0.5285 0 -> xyz=0.15 0 0

Commit message: Update test_design.urdf

File: r3ros/urdf/test_design.urdf (robot description, URDF)
Before this commit: robot cougarbot, 5 links, 4 joints
Joints:
- joint front_left_wheelconnect: origin xyz=0 0 0 -> xyz=0.15 0 0

Commit message: Update test_design.urdf

File: r3ros/urdf/test_design.urdf (robot description, URDF)
Before this commit: robot cougarbot, 5 links, 4 joints
Links:
- added link bl_wheel; visual cylinder length=0.050 radius=0.127
- added link ml_wheel; visual cylinder length=0.050 radius=0.127
Joints:
- added joint back_left_wheelconnect: type fixed, parent back_wheel_left_axel, child bl_wheel, origin xyz=0.15 0 0
- added joint middle_left_wheelconnect: type fixed, parent middle_wheel_left_axel, child ml_wheel, origin xyz=0.15 0 0

Commit message: Update test_design.urdf

File: r3ros/urdf/test_design.urdf (robot description, URDF)
Before this commit: robot cougarbot, 7 links, 6 joints
Links:
- added link back_wheel_right_axel; visual box size=0.3 .1 0.06
- added link front_wheel_right_axel; visual box size=0.3 .1 0.06
- added link middle_wheel_right_axel; visual box size=0.3 .1 0.06
Joints:
- added joint back_right_jointconnect: type fixed, parent base_link, child back_wheel_right_axel, origin xyz=0.15 0.5285 0
- added joint front_right_jointconnect: type fixed, parent base_link, child front_wheel_right_axel, origin xyz=0.15 -0.5285 0
- added joint middle_right_jointconnect: type fixed, parent base_link, child middle_wheel_right_axel, origin xyz=0.15 0 0

Commit message: Update test_design.urdf

File: r3ros/urdf/test_design.urdf (robot description, URDF)
Before this commit: robot cougarbot, 10 links, 9 joints
Joints:
- joint back_right_jointconnect: origin xyz=0.15 0.5285 0 -> xyz=-0.15 0.5285 0
- joint front_right_jointconnect: origin xyz=0.15 -0.5285 0 -> xyz=-0.15 -0.5285 0
- joint middle_right_jointconnect: origin xyz=0.15 0 0 -> xyz=-0.15 0 0

Commit message: Update test_design.urdf

File: r3ros/urdf/test_design.urdf (robot description, URDF)
Before this commit: robot cougarbot, 10 links, 9 joints
Links:
- added link br_wheel; visual cylinder length=0.050 radius=0.127
- added link fr_wheel; visual cylinder length=0.050 radius=0.127
- added link mr_wheel; visual cylinder length=0.050 radius=0.127
Joints:
- added joint back_right_wheelconnect: type fixed, parent back_wheel_right_axel, child br_wheel, origin xyz=-0.3 0 0
- added joint front_right_wheelconnect: type fixed, parent front_wheel_right_axel, child fr_wheel, origin xyz=-0.3 0 0
- added joint middle_right_wheelconnect: type fixed, parent middle_wheel_right_axel, child mr_wheel, origin xyz=-0.3 0 0
- joint back_left_wheelconnect: origin xyz=0.15 0 0 -> xyz=0.3 0 0
- joint front_left_wheelconnect: origin xyz=0.15 0 0 -> xyz=0.3 0 0
- joint middle_left_wheelconnect: origin xyz=0.15 0 0 -> xyz=0.3 0 0

Commit message: Update test_design.urdf

File: r3ros/urdf/test_design.urdf (robot description, URDF)
Before this commit: robot cougarbot, 13 links, 12 joints
Links:
- link bl_wheel: geometry visual cylinder length=0.10 radius=0.127
- link br_wheel: geometry visual cylinder length=0.10 radius=0.127
- link fl_wheel: geometry visual cylinder length=0.10 radius=0.127
- link fr_wheel: geometry visual cylinder length=0.10 radius=0.127
- link ml_wheel: geometry visual cylinder length=0.10 radius=0.127
- link mr_wheel: geometry visual cylinder length=0.10 radius=0.127

Commit message: Update test_design.urdf

File: r3ros/urdf/test_design.urdf (robot description, URDF)
Before this commit: robot cougarbot, 13 links, 12 joints
Joints:
- joint back_left_wheelconnect: type fixed -> continuous
- joint back_right_wheelconnect: type fixed -> continuous
- joint front_left_wheelconnect: type fixed -> continuous
- joint front_right_wheelconnect: type fixed -> continuous
- joint middle_left_wheelconnect: type fixed -> continuous
- joint middle_right_wheelconnect: type fixed -> continuous

Commit message: Update test_design.urdf

File: r3ros/urdf/test_design.urdf (robot description, URDF)
Before this commit: robot cougarbot, 13 links, 12 joints
Links:
- link base_link: mass None -> 1.0; geometry collision box size=0.16 1.057 0.12; visual box size=0.16 1.057 0.12

Commit message: Update test_design.urdf

File: r3ros/urdf/test_design.urdf (robot description, URDF)
Before this commit: robot cougarbot, 13 links, 12 joints
Links:
- link br_wheel: mass None -> 0.1; geometry collision cylinder length=0.1 radius=0.127; visual cylinder length=0.10 radius=0.127
- link fl_wheel: mass None -> 0.1; geometry collision cylinder length=0.1 radius=0.127; visual cylinder length=0.10 radius=0.127
- link fr_wheel: mass None -> 0.1; geometry collision cylinder length=0.1 radius=0.127; visual cylinder length=0.10 radius=0.127

Commit message: Update test_design.urdf

File: r3ros/urdf/test_design.urdf (robot description, URDF)
Before this commit: robot cougarbot, 13 links, 12 joints
Links:
- link bl_wheel: mass None -> 0.1; geometry collision cylinder length=0.1 radius=0.127; visual cylinder length=0.10 radius=0.127
- link ml_wheel: mass None -> 0.1; geometry collision cylinder length=0.1 radius=0.127; visual cylinder length=0.10 radius=0.127
- link mr_wheel: mass None -> 0.1; geometry collision cylinder length=0.1 radius=0.127; visual cylinder length=0.10 radius=0.127
Joints:
- joint front_right_wheelconnect: origin xyz=-0.3 0 0 -> xyz=-0.15 0 0
- joint middle_left_wheelconnect: origin xyz=0.3 0 0 -> xyz=0.15 0 0

Commit message: Update test_design.urdf

File: r3ros/urdf/test_design.urdf (robot description, URDF)
Before this commit: robot cougarbot, 13 links, 12 joints
Joints:
- joint back_left_wheelconnect: axis (none) -> 0 0 1
- joint back_right_wheelconnect: axis (none) -> 0 0 1
- joint front_left_wheelconnect: axis (none) -> 0 0 1
- joint front_right_wheelconnect: axis (none) -> 0 0 1
- joint middle_left_wheelconnect: axis (none) -> 0 0 1
- joint middle_right_wheelconnect: axis (none) -> 0 0 1

Commit message: Update test_design.urdf

File: r3ros/urdf/test_design.urdf (robot description, URDF)
Before this commit: robot cougarbot, 13 links, 12 joints
Links:
- added link left_wheel, mass 0.1; collision cylinder length=0.05 radius=0.035; visual cylinder length=0.05 radius=0.035
Joints:
- added joint left_wheel_joint: type continuous, parent base_link, child left_wheel, origin xyz=-0.2825 0.125 -.15 rpy=-1.5708 0 0, axis 0 0 1

Commit message: Update test_design.urdf

File: r3ros/urdf/test_design.urdf (robot description, URDF)
Before this commit: robot cougarbot, 14 links, 13 joints
Joints:
- joint middle_right_wheelconnect: parent middle_wheel_right_axel -> base_link

Commit message: Update test_design.urdf

File: r3ros/urdf/test_design.urdf (robot description, URDF)
Before this commit: robot cougarbot, 14 links, 13 joints
Links:
- removed link left_wheel
Joints:
- removed joint left_wheel_joint
- joint back_left_wheelconnect: parent back_wheel_left_axel -> base_link
- joint back_right_wheelconnect: parent back_wheel_right_axel -> base_link
- joint front_left_wheelconnect: parent front_wheel_left_axel -> base_link
- joint front_right_wheelconnect: origin xyz=-0.15 0 0 -> xyz=-0.3 0 0; parent front_wheel_right_axel -> base_link
- joint middle_left_wheelconnect: origin xyz=0.15 0 0 -> xyz=0.3 0 0; parent middle_wheel_left_axel -> base_link

Commit message: Update test_design.urdf

File: r3ros/urdf/test_design.urdf (robot description, URDF)
Before this commit: robot cougarbot, 13 links, 12 joints
Joints:
- joint back_left_wheelconnect: axis 0 0 1 -> 0 1 0; origin xyz=0.3 0 0 -> xyz=0.3 -0.5285 0
- joint back_right_wheelconnect: axis 0 0 1 -> 0 1 0; origin xyz=-0.3 0 0 -> xyz=-0.3 -0.5285 0
- joint front_left_wheelconnect: axis 0 0 1 -> 0 1 0; origin xyz=0.3 0 0 -> xyz=0.3 0.5285 0
- joint front_right_wheelconnect: axis 0 0 1 -> 0 1 0; origin xyz=-0.3 0 0 -> xyz=-0.3 0.5285 0
- joint middle_left_wheelconnect: axis 0 0 1 -> 0 1 0; origin xyz=0.3 0 0 -> xyz=0.3 0.5285 0
- joint middle_right_wheelconnect: axis 0 0 1 -> 0 1 0

Commit message: Update test_design.urdf

File: r3ros/urdf/test_design.urdf (robot description, URDF)
Before this commit: robot cougarbot, 13 links, 12 joints
Joints:
- joint back_left_wheelconnect: axis 0 1 0 -> 1 0 0
- joint back_right_wheelconnect: axis 0 1 0 -> 1 0 0
- joint front_left_wheelconnect: axis 0 1 0 -> 1 0 0
- joint front_right_wheelconnect: axis 0 1 0 -> 1 0 0
- joint middle_left_wheelconnect: axis 0 1 0 -> 1 0 0; origin xyz=0.3 0.5285 0 -> xyz=0.3 0 0
- joint middle_right_wheelconnect: axis 0 1 0 -> 1 0 0

Commit message: Update test_design.urdf

File: r3ros/urdf/test_design.urdf (robot description, URDF)
Before this commit: robot cougarbot, 13 links, 12 joints
Joints:
- joint back_left_jointconnect: origin xyz=0.15 0.5285 0 -> xyz=0.15 0.5285 2
- joint back_left_wheelconnect: origin xyz=0.3 -0.5285 0 -> xyz=0.3 -0.5285 2
- joint back_right_jointconnect: origin xyz=-0.15 0.5285 0 -> xyz=-0.15 0.5285 2
- joint back_right_wheelconnect: origin xyz=-0.3 -0.5285 0 -> xyz=-0.3 -0.5285 2
- joint front_left_jointconnect: origin xyz=0.15 -0.5285 0 -> xyz=0.15 -0.5285 2
- joint front_left_wheelconnect: origin xyz=0.3 0.5285 0 -> xyz=0.3 0.5285 2
- joint front_right_jointconnect: origin xyz=-0.15 -0.5285 0 -> xyz=-0.15 -0.5285 2
- joint front_right_wheelconnect: origin xyz=-0.3 0.5285 0 -> xyz=-0.3 0.5285 2
- joint middle_left_jointconnect: origin xyz=0.15 0 0 -> xyz=0.15 0 2
- joint middle_left_wheelconnect: origin xyz=0.3 0 0 -> xyz=0.3 0 2
- joint middle_right_jointconnect: origin xyz=-0.15 0 0 -> xyz=-0.15 0 2
- joint middle_right_wheelconnect: origin xyz=-0.3 0 0 -> xyz=-0.3 0 2

Commit message: Revert "Update test_design.urdf"
This reverts commit 503fa29b85eaca849bb5367641bf8442fa192827.

File: r3ros/urdf/test_design.urdf (robot description, URDF)
Before this commit: robot cougarbot, 13 links, 12 joints
Joints:
- joint back_left_jointconnect: origin xyz=0.15 0.5285 2 -> xyz=0.15 0.5285 0
- joint back_left_wheelconnect: origin xyz=0.3 -0.5285 2 -> xyz=0.3 -0.5285 0
- joint back_right_jointconnect: origin xyz=-0.15 0.5285 2 -> xyz=-0.15 0.5285 0
- joint back_right_wheelconnect: origin xyz=-0.3 -0.5285 2 -> xyz=-0.3 -0.5285 0
- joint front_left_jointconnect: origin xyz=0.15 -0.5285 2 -> xyz=0.15 -0.5285 0
- joint front_left_wheelconnect: origin xyz=0.3 0.5285 2 -> xyz=0.3 0.5285 0
- joint front_right_jointconnect: origin xyz=-0.15 -0.5285 2 -> xyz=-0.15 -0.5285 0
- joint front_right_wheelconnect: origin xyz=-0.3 0.5285 2 -> xyz=-0.3 0.5285 0
- joint middle_left_jointconnect: origin xyz=0.15 0 2 -> xyz=0.15 0 0
- joint middle_left_wheelconnect: origin xyz=0.3 0 2 -> xyz=0.3 0 0
- joint middle_right_jointconnect: origin xyz=-0.15 0 2 -> xyz=-0.15 0 0
- joint middle_right_wheelconnect: origin xyz=-0.3 0 2 -> xyz=-0.3 0 0

Commit message: Update test_design.urdf

File: r3ros/urdf/test_design.urdf (robot description, URDF)
Before this commit: robot cougarbot, 13 links, 12 joints
Joints:
- joint middle_right_wheelconnect: origin xyz=-0.3 0 0 -> xyz=-0.3 0 .5

Commit message: Update test_design.urdf

File: r3ros/urdf/test_design.urdf (robot description, URDF)
Before this commit: robot cougarbot, 13 links, 12 joints
Joints:
- joint back_left_wheelconnect: origin xyz=0.3 -0.5285 0 -> xyz=0.3 -0.5285 0.12
- joint back_right_wheelconnect: origin xyz=-0.3 -0.5285 0 -> xyz=-0.3 -0.5285 .12
- joint front_left_wheelconnect: origin xyz=0.3 0.5285 0 -> xyz=0.3 0.5285 0.12
- joint front_right_wheelconnect: origin xyz=-0.3 0.5285 0 -> xyz=-0.3 0.5285 0.12
- joint middle_left_wheelconnect: origin xyz=0.3 0 0 -> xyz=0.3 0 0.12
- joint middle_right_wheelconnect: origin xyz=-0.3 0 .5 -> xyz=-0.3 0 .12

Commit message: Update test_design.urdf

File: r3ros/urdf/test_design.urdf (robot description, URDF)
Before this commit: robot cougarbot, 13 links, 12 joints
Joints:
- joint back_left_jointconnect: origin xyz=0.15 0.5285 0 -> xyz=0.15 0.5285 0.12
- joint back_right_jointconnect: origin xyz=-0.15 0.5285 0 -> xyz=-0.15 0.5285 0.12
- joint front_left_jointconnect: origin xyz=0.15 -0.5285 0 -> xyz=0.15 -0.5285 0.12
- joint front_right_jointconnect: origin xyz=-0.15 -0.5285 0 -> xyz=-0.15 -0.5285 0.12
- joint middle_left_jointconnect: origin xyz=0.15 0 0 -> xyz=0.15 0 0.12
- joint middle_right_jointconnect: origin xyz=-0.15 0 0 -> xyz=-0.15 0 0.12

Commit message: Update test_design.urdf

File: r3ros/urdf/test_design.urdf (robot description, URDF)
Before this commit: robot cougarbot, 13 links, 12 joints
Links:
- link base_link: geometry collision box size=0.16 1.057 0.12; visual box size=0.16 1.057 0.06

Commit message: Update test_design.urdf

File: r3ros/urdf/test_design.urdf (robot description, URDF)
Before this commit: robot cougarbot, 13 links, 12 joints
Joints:
- joint middle_right_jointconnect: origin xyz=-0.15 0 0.12 -> xyz=-0.15 0 0.08
- joint middle_right_wheelconnect: origin xyz=-0.3 0 .12 -> xyz=-0.3 0 .08

Commit message: Update test_design.urdf

File: r3ros/urdf/test_design.urdf (robot description, URDF)
Before this commit: robot cougarbot, 13 links, 12 joints
Joints:
- joint back_left_jointconnect: origin xyz=0.15 0.5285 0.12 -> xyz=0.15 0.5285 0
- joint back_left_wheelconnect: origin xyz=0.3 -0.5285 0.12 -> xyz=0.3 -0.5285 0
- joint back_right_jointconnect: origin xyz=-0.15 0.5285 0.12 -> xyz=-0.15 0.5285 0
- joint back_right_wheelconnect: origin xyz=-0.3 -0.5285 .12 -> xyz=-0.3 -0.5285 0
- joint front_left_jointconnect: origin xyz=0.15 -0.5285 0.12 -> xyz=0.15 -0.5285 0
- joint front_left_wheelconnect: origin xyz=0.3 0.5285 0.12 -> xyz=0.3 0.5285 0
- joint front_right_jointconnect: origin xyz=-0.15 -0.5285 0.12 -> xyz=-0.15 -0.5285 0
- joint front_right_wheelconnect: origin xyz=-0.3 0.5285 0.12 -> xyz=-0.3 0.5285 0
- joint middle_left_jointconnect: origin xyz=0.15 0 0.12 -> xyz=0.15 0 0
- joint middle_left_wheelconnect: origin xyz=0.3 0 0.12 -> xyz=0.3 0 0
- joint middle_right_jointconnect: origin xyz=-0.15 0 0.08 -> xyz=-0.15 0 0
- joint middle_right_wheelconnect: origin xyz=-0.3 0 .08 -> xyz=-0.3 0 0

Commit message: Update test_design.urdf

File: r3ros/urdf/test_design.urdf (robot description, URDF)
Before this commit: robot cougarbot, 13 links, 12 joints
Links:
- link base_link: geometry collision box size=0.508 1.057 0.12; visual box size=0.508 1.057 0.06
