Commit message: Joint Limits

File: devstuff/r3ros/arm-urdf/arm.urdf (robot description, URDF)
Before this commit: robot URC, 9 links, 8 joints
Links:
- link base_link: geometry collision cylinder length=0.05 radius=0.1; visual cylinder length=0.0 radius=0.05
- link grip_finger: geometry collision box size=0.22 0.1 0.22; visual box size=0.03 0.1 0.08
- link grip_fixed: geometry collision box size=0.22 0.1 0.22; visual box size=0.03 0.1 0.08
Joints:
- joint base_twist: origin xyz=0.0 0.0 0.05 rpy=0 0 0 -> xyz=0.0 0.0 0.0 rpy=0 0 0
- joint elbow_lower: limit (none) -> lower=0.698 upper=-1.396 effort=30 velocity=1.0; type continuous -> revolute
- joint elbow_middle: limit (none) -> lower=2.96706 upper=1.31 effort=1000.0 velocity=0.5; type continuous -> revolute
- joint elbow_upper: limit (none) -> lower=-2.00713 upper=2.00713 effort=1000.0 velocity=0.5; type continuous -> revolute
- joint grip: limit lower=-0.38 upper=0 effort=1000.0 velocity=0.5 -> lower=-0.175 upper=0 effort=1000.0 velocity=0.5; origin xyz=0.0 0.0 0.2525 rpy=0 0 1.57075 -> xyz=0.0 0.075 0.09125 rpy=0 0 1.57075
- joint grip_base_to_fixed: origin xyz=0.0 0.0 0.01525 rpy=0 0 0 -> xyz=0.0 0.096 0.09125 rpy=0 0 1.57075
