Commit message: Few things:
Finish protocol docs for the arm code
Correct weight values in the urdf
Almost finish the actual actionserver code in python

File: rosws/src/rover_arm/arm.urdf (robot description, URDF)
Before this commit: robot arm, 9 links, 8 joints
Links:
- link base_link: mass 1.0 -> 0.5
- link grip_finger: mass 1.0 -> 0.25
- link hand: mass 1.0 -> 0.25
- link lower_arm: mass 1.0 -> 0.5
- link middle_arm: mass 1.0 -> 0.5
- link torso: mass 1.0 -> 0.5
- link upper_arm: mass 1.0 -> 0.5

Commit message: More realistic joint rotation limits

File: rosws/src/rover_arm/arm.urdf (robot description, URDF)
Before this commit: robot arm, 9 links, 8 joints
Joints:
- joint elbow: limit (none) -> lower=0 upper=2.5 effort=1000 velocity=10.0; type continuous -> revolute
- joint hip: limit (none) -> effort=1000 velocity=10.0
- joint lower_elbow: limit (none) -> lower=-1.9 upper=1.9 effort=1000 velocity=10.0; type continuous -> revolute
- joint shoulder: limit (none) -> lower=-1.57 upper=0.1 effort=1000 velocity=10.0; type continuous -> revolute
- joint wrist: limit (none) -> effort=1000 velocity=10.0

Commit message: Slow down arm movement speed

File: rosws/src/rover_arm/arm.urdf (robot description, URDF)
Before this commit: robot arm, 9 links, 8 joints
Joints:
- joint elbow: limit lower=0 upper=2.5 effort=1000 velocity=10.0 -> lower=0 upper=2.5 effort=1000 velocity=0.1
- joint hip: limit effort=1000 velocity=10.0 -> effort=1000 velocity=0.1
- joint lower_elbow: limit lower=-1.9 upper=1.9 effort=1000 velocity=10.0 -> lower=-1.9 upper=1.9 effort=1000 velocity=0.1
- joint shoulder: limit lower=-1.57 upper=0.1 effort=1000 velocity=10.0 -> lower=-1.57 upper=0.1 effort=1000 velocity=0.1
- joint wrist: limit effort=1000 velocity=10.0 -> effort=1000 velocity=0.1
